Commit message: Publishing best estimation for the nested pose and visualize it using TF

File: robots/boxes/box_green.urdf.xacro (robot description, xacro)
@@ -19,5 +19,5 @@
       </visual>
   	  <collision>
-        <origin xyz="0.0 0.0 0.0" rpy="0 0 0"/>
+        <origin xyz="0.0 0.0 0.0" rpy="0 0 ${M_PI/2}"/>
   	    <geometry>
   	      <box size="0.2 0.2 0.2"/>

File: robots/kobuki_hexagons_kinect_green.urdf.xacro (robot description, xacro)
@@ -8,7 +8,13 @@
   <xacro:include filename="$(find turtlebot_description)/urdf/turtlebot_library.urdf.xacro" />
   <xacro:include filename="$(find experiment_launcher)/robots/boxes/box_green.urdf.xacro" />
+  <xacro:include filename="$(find experiment_launcher)/robots/boxes/box_right.urdf.xacro" />
+  <xacro:include filename="$(find experiment_launcher)/robots/boxes/box_left.urdf.xacro" />
+  <xacro:include filename="$(find experiment_launcher)/robots/boxes/box_back.urdf.xacro" />
   <kobuki/>
   <stack_hexagons parent="base_link"/>
   <sensor_kinect  parent="base_link"/>
   <box_green	  parent="base_link"/>
+  <box_right	  parent="base_link"/>
+  <box_left 	  parent="base_link"/>
+  <box_back 	  parent="base_link"/>
 </robot>
