Commit message: Three robot experiment is ready

File: robots/boxes/box_back_white_big.urdf.xacro (robot description, xacro)
@@ -10,7 +10,7 @@
     <link name="box_back_link">
       <visual>
-       <origin xyz="-0.16 0.0 -0.2" rpy="0 0 0"/>
+       <origin xyz="-0.16 0.0 -0.1" rpy="0 0 0"/>
         <geometry>
-          <box size="0.01 0.3 0.3"/>
+          <box size="0.01 0.25 0.5"/>
         </geometry>
         <material name="white">
@@ -19,7 +19,7 @@
       </visual>
       <collision>
-        <origin xyz="-0.16 0.0 -0.2" rpy="0 0 0"/>
+        <origin xyz="-0.16 0.0 -0.1" rpy="0 0 0"/>
         <geometry>
-          <box size="0.01 0.3 0.3"/>
+          <box size="0.01 0.25 0.5"/>
         </geometry>
       </collision>

File: robots/kobuki_circles_kinect_covered.urdf.xacro (robot description, xacro)
@@ -7,4 +7,5 @@
 <robot name="turtlebot" xmlns:xacro="http://ros.org/wiki/xacro">
   <xacro:include filename="$(find turtlebot_description)/urdf/turtlebot_library.urdf.xacro" />
+  <xacro:include filename="$(find experiment_launcher)/robots/boxes/box_yellow.urdf.xacro" />
   <xacro:include filename="$(find experiment_launcher)/robots/boxes/box_right_white.urdf.xacro" />
   <xacro:include filename="$(find experiment_launcher)/robots/boxes/box_left_white.urdf.xacro" />
@@ -13,4 +14,5 @@
   <stack_circles parent="base_link"/>
   <sensor_kinect  parent="base_link"/>
+  <box_yellow    parent="base_link"/>
   <box_right	  parent="base_link"/>
   <box_left 	  parent="base_link"/>
